Commit message: fix(description): rename right wheel joint to Right_Wheel_Joint and correct rotation axis

File: ros_ws/src/REFLEX/reflex_descriptions/urdf/components/right_leg.xacro (robot description, xacro)
@@ -99,9 +99,9 @@
     </link>
     <!-- Right Wheel joint -->
-    <joint name="${prefix}Right_Wheel_Link" type="continuous">
+    <joint name="${prefix}Right_Wheel_Joint" type="continuous">
       <origin xyz="0.04 -0.2 0" rpy="1.5708 -0.91317 1.5708"/>
       <parent link="${prefix}Right_Knee"/>
       <child link="${prefix}Right_Wheel"/>
-      <axis xyz="0 0 1"/>
+      <axis xyz="0 0 -1"/>
     </joint>
   </xacro:macro>
