Commit message: feat(thirdPID): introduce third PID for stance control using vilocity

File: ros_ws/src/REFLEX/reflex_descriptions/urdf/components/left_leg.xacro (robot description, xacro)
@@ -34,6 +34,6 @@
       <child link="${prefix}Left_Hip"/>
       <!-- ! NOTE: SolidWorks exported axis="0 0 0" (invalid). Fix axis based on your hinge. -->
-      <axis xyz="0 0 1"/>
-      <limit lower="0" upper="0" effort="0" velocity="0"/>
+      <axis xyz="-1 0 0"/>
+      <limit lower="-1.5708" upper="1.5708" effort="11.0" velocity="43.98"/>
     </joint>
     <!-- Left Knee link -->
@@ -69,6 +69,6 @@
       <child link="${prefix}Left_Knee"/>
       <!-- ! NOTE: SolidWorks exported axis="0 0 0" (invalid). Fix axis based on your hinge. -->
-      <axis xyz="0 0 1"/>
-      <limit lower="0" upper="0" effort="0" velocity="0"/>
+      <axis xyz="-1 0 0"/>
+      <limit lower="-1.5708" upper="1.5708" effort="11.0" velocity="43.98"/>
     </joint>
     <!-- Left Wheel link -->
@@ -99,5 +99,5 @@
     </link>
     <!-- Left Wheel joint -->
-    <joint name="${prefix}Left_Wheel_Joint" type="continuous">
+    <joint name="${prefix}Left_Wheel_Joint" type="fixed">
       <origin xyz="0.04 -0.2 0" rpy="-1.5708 -0.91317 -1.5708"/>
       <parent link="${prefix}Left_Knee"/>

File: ros_ws/src/REFLEX/reflex_descriptions/urdf/components/right_leg.xacro (robot description, xacro)
@@ -35,5 +35,5 @@
       <axis xyz="1 0 0"/>
       <!-- NOTE: SolidWorks exported 0/0 limits. Replace with real joint limits. -->
-      <limit lower="0" upper="0" effort="0" velocity="0"/>
+      <limit lower="-1.5708" upper="1.5708" effort="11.0" velocity="43.98"/>
     </joint>
     <!-- Right Knee link -->
@@ -69,6 +69,6 @@
       <child link="${prefix}Right_Knee"/>
       <!-- ! NOTE: SolidWorks exported axis="0 0 0" (invalid). Fix axis based on your hinge. -->
-      <axis xyz="0 0 1"/>
-      <limit lower="0" upper="0" effort="0" velocity="0"/>
+      <axis xyz="1 0 0"/>
+      <limit lower="-1.5708" upper="1.5708" effort="11.0" velocity="43.98"/>
     </joint>
     <!-- Right Wheel link -->
@@ -99,5 +99,5 @@
     </link>
     <!-- Right Wheel joint -->
-    <joint name="${prefix}Right_Wheel_Joint" type="continuous">
+    <joint name="${prefix}Right_Wheel_Joint" type="fixed">
       <origin xyz="0.04 -0.2 0" rpy="1.5708 -0.91317 1.5708"/>
       <parent link="${prefix}Right_Knee"/>

File: ros_ws/src/REFLEX/reflex_descriptions/urdf/reflex.urdf.xacro (robot description, xacro)
@@ -14,3 +14,9 @@
   <xacro:reflex_right_leg prefix="${prefix}" parent="${prefix}base_link" />
   <!-- <xacro:reflex_sensors prefix="${prefix}" parent="${prefix}base_link" /> TODO: Add Sensors -->
+  <link name="world"/>
+  <joint name="test_stand_joint" type="fixed">
+    <origin xyz="0 0 1.0" rpy="0 0 0"/>
+    <parent link="world"/>
+    <child link="${prefix}base_link"/>
+  </joint>
 </robot>

File: ros_ws/src/REFLEX/reflex_gazebo/urdf/reflex_gazebo.xacro (robot description, xacro)
@@ -68,6 +68,5 @@
         <plugin>gz_ros2_control/GazeboSimSystem</plugin>
       </hardware>
-      <!-- Left wheel joint -->
-      <joint name="${prefix}Left_Wheel_Joint">
+      <joint name="${prefix}Left_Hip_joint">
         <command_interface name="velocity"/>
         <state_interface name="position"/>
@@ -75,6 +74,17 @@
         <state_interface name="effort"/>
       </joint>
-      <!-- Right wheel joint -->
-      <joint name="${prefix}Right_Wheel_Joint">
+      <joint name="${prefix}Left_Knee_joint">
+        <command_interface name="velocity"/>
+        <state_interface name="position"/>
+        <state_interface name="velocity"/>
+        <state_interface name="effort"/>
+      </joint>
+      <joint name="${prefix}Right_Hip_Joint">
+        <command_interface name="velocity"/>
+        <state_interface name="position"/>
+        <state_interface name="velocity"/>
+        <state_interface name="effort"/>
+      </joint>
+      <joint name="${prefix}Right_Knee_joint">
         <command_interface name="velocity"/>
         <state_interface name="position"/>

Commit message: feat(stance): Lower limits is set to -360 to 360 to be able to apply offsets

File: ros_ws/src/REFLEX/reflex_descriptions/urdf/components/left_leg.xacro (robot description, xacro)
@@ -35,5 +35,6 @@
       <!-- ! NOTE: SolidWorks exported axis="0 0 0" (invalid). Fix axis based on your hinge. -->
       <axis xyz="-1 0 0"/>
-      <limit lower="-1.5708" upper="1.5708" effort="11.0" velocity="43.98"/>
+      <!-- ! NOTE: Lower limits is set to -360 to 360 to be able to apply offsets -->
+      <limit lower="-3.14159" upper="3.14159" effort="11.0" velocity="43.98"/>
     </joint>
     <!-- Left Knee link -->
@@ -70,5 +71,6 @@
       <!-- ! NOTE: SolidWorks exported axis="0 0 0" (invalid). Fix axis based on your hinge. -->
       <axis xyz="-1 0 0"/>
-      <limit lower="-1.5708" upper="1.5708" effort="11.0" velocity="43.98"/>
+      <!-- ! NOTE: Lower limits is set to -360 to 360 to be able to apply offsets -->
+      <limit lower="-3.14159" upper="3.14159" effort="11.0" velocity="43.98"/>
     </joint>
     <!-- Left Wheel link -->

File: ros_ws/src/REFLEX/reflex_descriptions/urdf/components/right_leg.xacro (robot description, xacro)
@@ -35,5 +35,6 @@
       <axis xyz="1 0 0"/>
       <!-- NOTE: SolidWorks exported 0/0 limits. Replace with real joint limits. -->
-      <limit lower="-1.5708" upper="1.5708" effort="11.0" velocity="43.98"/>
+      <!-- ! NOTE: Lower limits is set to -360 to 360 to be able to apply offsets -->
+      <limit lower="-3.14159" upper="3.14159" effort="11.0" velocity="43.98"/>
     </joint>
     <!-- Right Knee link -->
@@ -70,5 +71,6 @@
       <!-- ! NOTE: SolidWorks exported axis="0 0 0" (invalid). Fix axis based on your hinge. -->
       <axis xyz="1 0 0"/>
-      <limit lower="-1.5708" upper="1.5708" effort="11.0" velocity="43.98"/>
+      <!-- ! NOTE: Lower limits is set to -360 to 360 to be able to apply offsets -->
+      <limit lower="-3.14159" upper="3.14159" effort="11.0" velocity="43.98"/>
     </joint>
     <!-- Right Wheel link -->

File: ros_ws/src/REFLEX/reflex_gazebo/models/reflex/model.urdf (robot description, URDF)
Before this commit: robot reflex, 7 links, 6 joints
Joints:
- joint Left_Hip_joint: limit lower=-1.5708 upper=1.5708 effort=11.0 velocity=43.98 -> lower=-3.14159 upper=3.14159 effort=11.0 velocity=43.98
- joint Left_Knee_joint: limit lower=-1.5708 upper=1.5708 effort=11.0 velocity=43.98 -> lower=-3.14159 upper=3.14159 effort=11.0 velocity=43.98
- joint Right_Hip_Joint: limit lower=-1.5708 upper=1.5708 effort=11.0 velocity=43.98 -> lower=-3.14159 upper=3.14159 effort=11.0 velocity=43.98
- joint Right_Knee_joint: limit lower=-1.5708 upper=1.5708 effort=11.0 velocity=43.98 -> lower=-3.14159 upper=3.14159 effort=11.0 velocity=43.98

Commit message: feat(stance): reverse Knee angle direction in both legs

File: ros_ws/src/REFLEX/reflex_descriptions/urdf/components/left_leg.xacro (robot description, xacro)
@@ -70,5 +70,5 @@
       <child link="${prefix}Left_Knee"/>
       <!-- ! NOTE: SolidWorks exported axis="0 0 0" (invalid). Fix axis based on your hinge. -->
-      <axis xyz="-1 0 0"/>
+      <axis xyz="1 0 0"/>
       <!-- ! NOTE: Lower limits is set to -360 to 360 to be able to apply offsets -->
       <limit lower="-3.14159" upper="3.14159" effort="11.0" velocity="43.98"/>
@@ -101,5 +101,5 @@
     </link>
     <!-- Left Wheel joint -->
-    <joint name="${prefix}Left_Wheel_Joint" type="fixed">
+    <joint name="${prefix}Left_Wheel_Joint" type="continuous">
       <origin xyz="0.04 -0.2 0" rpy="-1.5708 -0.91317 -1.5708"/>
       <parent link="${prefix}Left_Knee"/>

File: ros_ws/src/REFLEX/reflex_descriptions/urdf/components/right_leg.xacro (robot description, xacro)
@@ -70,5 +70,5 @@
       <child link="${prefix}Right_Knee"/>
       <!-- ! NOTE: SolidWorks exported axis="0 0 0" (invalid). Fix axis based on your hinge. -->
-      <axis xyz="1 0 0"/>
+      <axis xyz="-1 0 0"/>
       <!-- ! NOTE: Lower limits is set to -360 to 360 to be able to apply offsets -->
       <limit lower="-3.14159" upper="3.14159" effort="11.0" velocity="43.98"/>
@@ -101,5 +101,5 @@
     </link>
     <!-- Right Wheel joint -->
-    <joint name="${prefix}Right_Wheel_Joint" type="fixed">
+    <joint name="${prefix}Right_Wheel_Joint" type="continuous">
       <origin xyz="0.04 -0.2 0" rpy="1.5708 -0.91317 1.5708"/>
       <parent link="${prefix}Right_Knee"/>
