Commit message: feat(stance): fix controller's name

File: ros_ws/src/REFLEX/reflex_gazebo/models/reflex/model.urdf (robot description, URDF)
Before this commit: robot reflex, 7 links, 6 joints
Joints:
- joint Left_Hip_joint: axis 0 0 1 -> -1 0 0; limit lower=0 upper=0 effort=0 velocity=0 -> lower=-1.5708 upper=1.5708 effort=11.0 velocity=43.98
- joint Left_Knee_joint: axis 0 0 1 -> -1 0 0; limit lower=0 upper=0 effort=0 velocity=0 -> lower=-1.5708 upper=1.5708 effort=11.0 velocity=43.98
- joint Left_Wheel_Joint: type continuous -> fixed
- joint Right_Hip_Joint: limit lower=0 upper=0 effort=0 velocity=0 -> lower=-1.5708 upper=1.5708 effort=11.0 velocity=43.98
- joint Right_Knee_joint: axis 0 0 1 -> 1 0 0; limit lower=0 upper=0 effort=0 velocity=0 -> lower=-1.5708 upper=1.5708 effort=11.0 velocity=43.98
- joint Right_Wheel_Joint: type continuous -> fixed

Commit message: feat(stance): release the wheel joints and merge the roll balance branch

File: ros_ws/src/REFLEX/reflex_gazebo/models/reflex/model.urdf (robot description, URDF)
Before this commit: robot reflex, 7 links, 6 joints
Joints:
- joint Left_Knee_joint: axis -1 0 0 -> 1 0 0
- joint Left_Wheel_Joint: type fixed -> continuous
- joint Right_Knee_joint: axis 1 0 0 -> -1 0 0
- joint Right_Wheel_Joint: type fixed -> continuous
