Commit message: feat(stance): Add wheels command interface and states

File: ros_ws/src/REFLEX/reflex_gazebo/urdf/reflex_gazebo.xacro (robot description, xacro)
@@ -80,4 +80,10 @@
         <state_interface name="effort"/>
       </joint>
+            <joint name="${prefix}Left_Wheel_Joint">
+        <command_interface name="velocity"/>
+        <state_interface name="position"/>
+        <state_interface name="velocity"/>
+        <state_interface name="effort"/>
+      </joint>
       <joint name="${prefix}Right_Hip_Joint">
         <command_interface name="velocity"/>
@@ -87,4 +93,10 @@
       </joint>
       <joint name="${prefix}Right_Knee_joint">
+        <command_interface name="velocity"/>
+        <state_interface name="position"/>
+        <state_interface name="velocity"/>
+        <state_interface name="effort"/>
+      </joint>
+      <joint name="${prefix}Right_Wheel_Joint">
         <command_interface name="velocity"/>
         <state_interface name="position"/>
