Commit message: feat(stance): change how we fix robot base link to world

File: ros_ws/src/REFLEX/reflex_descriptions/urdf/reflex.urdf.xacro (robot description, xacro)
@@ -14,9 +14,3 @@
   <xacro:reflex_right_leg prefix="${prefix}" parent="${prefix}base_link" />
   <!-- <xacro:reflex_sensors prefix="${prefix}" parent="${prefix}base_link" /> TODO: Add Sensors -->
-  <link name="world"/>
-  <joint name="test_stand_joint" type="fixed">
-    <origin xyz="0 0 1.0" rpy="0 0 0"/>
-    <parent link="world"/>
-    <child link="${prefix}base_link"/>
-  </joint>
 </robot>

Commit message: feat(stance): add dummy link so base_link doesn't have inertia

File: ros_ws/src/REFLEX/reflex_descriptions/urdf/reflex.urdf.xacro (robot description, xacro)
@@ -10,5 +10,11 @@
   <!-- <xacro:include filename="$(find reflex_descriptions)/urdf/components/sensors.xacro" /> TODO: Add sensors -->
   <!-- Build robot -->
+  <link name="${prefix}base_root"/>
   <xacro:reflex_base prefix="${prefix}" />
+  <joint name="${prefix}base_root_joint" type="fixed">
+    <parent link="${prefix}base_root" />
+    <child link="${prefix}base_link" />
+    <origin xyz="0 0 0" rpy="0 0 0" />
+  </joint>
   <xacro:reflex_left_leg prefix="${prefix}" parent="${prefix}base_link" />
   <xacro:reflex_right_leg prefix="${prefix}" parent="${prefix}base_link" />

File: ros_ws/src/REFLEX/reflex_gazebo/models/reflex/model.urdf (robot description, URDF)
Before this commit: robot reflex, 7 links, 6 joints
Links:
- added link base_root
Joints:
- added joint base_root_joint: type fixed, parent base_root, child base_link, origin xyz=0 0 0 rpy=0 0 0
